Commit message: Model dispenser and gripper occupancy conservatively
Merge the four measured nozzle/head boxes into one upright cuboid so the empty gaps between outlets are also treated as occupied during planning review. Add a link_6-attached RG2-style collision envelope so MoveIt previews no longer assume an empty flange.

Constraint: Do not invent cup coordinates or measured calibration values; derive nozzle span only from existing measured nozzle boxes and keep real-motion enable flags false.
Rejected: Keeping four tilted nozzle boxes | it left gaps and orientation artifacts the operator explicitly wanted removed.
Confidence: high
Scope-risk: moderate
Directive: Keep the gripper envelope synchronized with rg2_link6_tcp.urdf.xacro if dimensions change.
Tested: python3 -m py_compile for changed Python/launch files; YAML merged-block assertion; xacro rg2_link6_tcp.urdf.xacro; colcon build --packages-select azas_motion azas_bringup --symlink-install; ros2 run azas_motion link6_gripper_collision_node --ros-args -p publish_once:=true; ros2 launch azas_bringup rg2_link6_tcp.launch.py --show-args; python3 tools/checks/check_measured_dispenser_geometry.py
Not-tested: live robot motion and physical collision clearance.

File: src/azas_bringup/urdf/rg2_link6_tcp.urdf.xacro (robot description, xacro)
@@ -5,4 +5,7 @@
   <material name="azas_rg2_dark">
     <color rgba="0.08 0.08 0.09 1.0"/>
+  </material>
+  <material name="azas_rg2_metal">
+    <color rgba="0.42 0.43 0.45 1.0"/>
   </material>
   <material name="azas_rg2_tip">
@@ -24,14 +27,27 @@
   <link name="GripperDA_v1_jarvis">
     <visual>
-      <origin xyz="0 0 0.055" rpy="0 0 0"/>
+      <origin xyz="0 0 0.025" rpy="0 0 0"/>
       <geometry>
-        <box size="0.080 0.055 0.110"/>
+        <cylinder radius="0.040" length="0.050"/>
+      </geometry>
+      <material name="azas_rg2_metal"/>
+    </visual>
+    <visual>
+      <origin xyz="0 0 0.075" rpy="0 0 0"/>
+      <geometry>
+        <box size="0.090 0.140 0.050"/>
       </geometry>
       <material name="azas_rg2_dark"/>
     </visual>
     <collision>
-      <origin xyz="0 0 0.055" rpy="0 0 0"/>
+      <origin xyz="0 0 0.025" rpy="0 0 0"/>
       <geometry>
-        <box size="0.080 0.055 0.110"/>
+        <cylinder radius="0.040" length="0.050"/>
+      </geometry>
+    </collision>
+    <collision>
+      <origin xyz="0 0 0.075" rpy="0 0 0"/>
+      <geometry>
+        <box size="0.090 0.140 0.050"/>
       </geometry>
     </collision>
@@ -40,18 +56,31 @@
     <parent link="GripperDA_v1_jarvis"/>
     <child link="rg2_left_finger_visual"/>
-    <origin xyz="0 0.035 0.145" rpy="0 0 0"/>
+    <origin xyz="0 0.055 0.155" rpy="0 0 0"/>
   </joint>
   <link name="rg2_left_finger_visual">
     <visual>
-      <origin xyz="0 0 0.040" rpy="0 0 0"/>
+      <origin xyz="0 0 0" rpy="0 0 0"/>
       <geometry>
-        <box size="0.020 0.018 0.080"/>
+        <box size="0.035 0.018 0.160"/>
+      </geometry>
+      <material name="azas_rg2_dark"/>
+    </visual>
+    <visual>
+      <origin xyz="0 -0.015 0.090" rpy="0 0 0"/>
+      <geometry>
+        <box size="0.025 0.012 0.035"/>
       </geometry>
       <material name="azas_rg2_tip"/>
     </visual>
     <collision>
-      <origin xyz="0 0 0.040" rpy="0 0 0"/>
+      <origin xyz="0 0 0" rpy="0 0 0"/>
       <geometry>
-        <box size="0.020 0.018 0.080"/>
+        <box size="0.035 0.018 0.160"/>
+      </geometry>
+    </collision>
+    <collision>
+      <origin xyz="0 -0.015 0.090" rpy="0 0 0"/>
+      <geometry>
+        <box size="0.025 0.012 0.035"/>
       </geometry>
     </collision>
@@ -60,18 +89,31 @@
     <parent link="GripperDA_v1_jarvis"/>
     <child link="rg2_right_finger_visual"/>
-    <origin xyz="0 -0.035 0.145" rpy="0 0 0"/>
+    <origin xyz="0 -0.055 0.155" rpy="0 0 0"/>
   </joint>
   <link name="rg2_right_finger_visual">
     <visual>
-      <origin xyz="0 0 0.040" rpy="0 0 0"/>
+      <origin xyz="0 0 0" rpy="0 0 0"/>
       <geometry>
-        <box size="0.020 0.018 0.080"/>
+        <box size="0.035 0.018 0.160"/>
+      </geometry>
+      <material name="azas_rg2_dark"/>
+    </visual>
+    <visual>
+      <origin xyz="0 0.015 0.090" rpy="0 0 0"/>
+      <geometry>
+        <box size="0.025 0.012 0.035"/>
       </geometry>
       <material name="azas_rg2_tip"/>
     </visual>
     <collision>
-      <origin xyz="0 0 0.040" rpy="0 0 0"/>
+      <origin xyz="0 0 0" rpy="0 0 0"/>
       <geometry>
-        <box size="0.020 0.018 0.080"/>
+        <box size="0.035 0.018 0.160"/>
+      </geometry>
+    </collision>
+    <collision>
+      <origin xyz="0 0.015 0.090" rpy="0 0 0"/>
+      <geometry>
+        <box size="0.025 0.012 0.035"/>
       </geometry>
     </collision>
